Commit message: fixed rviz2 being too fast

File: description/lidar.xacro (robot description, xacro)
@@ -29,5 +29,5 @@
             <pose>0 0 0 0 0 0</pose>
             <visualize>true</visualize>
-            <update_rate>10</update_rate>
+            <update_rate>30</update_rate>
             <ray>
                 <scan>
@@ -47,5 +47,5 @@
             <plugin name="laser_controller" filename="libgazebo_ros_ray_sensor.so">
                 <ros>
-                    <argument>-/out:=scan</argument>
+                    <argument>~/out:=scan</argument>
                 </ros>
                 <output_type>sensor_msgs/LaserScan</output_type>

File: description/robot.urdf.xacro (robot description, xacro)
@@ -2,6 +2,6 @@
 <robot xmlns:xacro="http://www.ros.org/wiki/xacro"  name="robot">
     <xacro:include filename="robot_core.xacro"/>
-    <xacro:include filename="gazebo_control.xacro"/>
-    <!-- <xacro:include filename="ros2_control.xacro"/> -->
+    <!-- <xacro:include filename="gazebo_control.xacro"/> -->
+    <xacro:include filename="ros2_control.xacro"/>
     <xacro:include filename="lidar.xacro"/>
 </robot>

File: description/robot_core.xacro (robot description, xacro)
@@ -56,4 +56,5 @@
     <link name="left_wheel">
         <visual>
+            <origin xyz="0 0 0"/>
             <geometry>
                 <cylinder radius="0.0325" length="0.026"/>
@@ -62,9 +63,10 @@
         </visual>
         <collision>
+            <origin xyz="0 0 0"/>
             <geometry>
-                <cylinder radius="0.0325" length="0.026"/>
+                <sphere radius="0.0325"/>
             </geometry>
         </collision>
-        <xacro:inertial_cylinder mass= "0.1" radius="0.125" length="0.026">
+        <xacro:inertial_cylinder mass= "0.1" radius="0.0325" length="0.026">
             <origin xyz="0.0 0.0 0.0" rpy="0.0 0.0 0.0"/>
         </xacro:inertial_cylinder>
@@ -82,4 +84,5 @@
     <link name="right_wheel">
         <visual>
+            <origin xyz="0 0 0"/>
             <geometry>
                 <cylinder radius="0.0325" length="0.026"/>
@@ -88,9 +91,10 @@
         </visual>
         <collision>
+            <origin xyz="0 0 0"/>
             <geometry>
-                <cylinder radius="0.0325" length="0.026"/>
+                <sphere radius="0.0325"/>
             </geometry>
         </collision>
-        <xacro:inertial_cylinder mass= "0.1" radius="0.125" length="0.026">
+        <xacro:inertial_cylinder mass= "0.1" radius="0.0325" length="0.026">
             <origin xyz="0.0 0.0 0.0" rpy="0.0 0.0 0.0"/>
         </xacro:inertial_cylinder>
@@ -107,4 +111,5 @@
     <link name="front_castor_wheel">
         <visual>
+            <origin xyz="0 0 0"/>
             <geometry>
                 <sphere radius="0.0325"/>
@@ -113,9 +118,10 @@
         </visual>
         <collision>
+            <origin xyz="0 0 0"/>
             <geometry>
                 <sphere radius="0.0325"/>
             </geometry>
         </collision>
-        <xacro:inertial_sphere mass= "0.1" radius="0.325">
+        <xacro:inertial_sphere mass= "0.1" radius="0.0325">
             <origin xyz="0.0 0.0 0.0" rpy="0.0 0.0 0.0"/>
         </xacro:inertial_sphere>
@@ -134,4 +140,5 @@
     <link name="back_castor_wheel">
         <visual>
+            <origin xyz="0 0 0"/>
             <geometry>
                 <sphere radius="0.0325"/>
@@ -140,9 +147,10 @@
         </visual>
         <collision>
+            <origin xyz="0 0 0"/>
             <geometry>
                 <sphere radius="0.0325"/>
             </geometry>
         </collision>
-        <xacro:inertial_sphere mass= "0.1" radius="0.325">
+        <xacro:inertial_sphere mass= "0.1" radius="0.0325">
             <origin xyz="0.0 0.0 0.0" rpy="0.0 0.0 0.0"/>
         </xacro:inertial_sphere>
