Commit message: added ros control

File: description/robot.urdf.xacro (robot description, xacro)
@@ -3,3 +3,5 @@
     <xacro:include filename="robot_core.xacro"/>
     <xacro:include filename="gazebo_control.xacro"/>
+    <!-- <xacro:include filename="ros2_control.xacro"/> -->
+    <xacro:include filename="lidar.xacro"/>
 </robot>

File: description/robot_core.xacro (robot description, xacro)
@@ -13,4 +13,7 @@
     <material name = "black">
         <color rgba = "0 0 0 1"/>
+    </material>
+    <material name = "red">
+        <color rgba = "1 0 0 1"/>
     </material>
     <!-- base link -->

Commit message: Added slam toolbox

File: description/robot.urdf.xacro (robot description, xacro)
@@ -1,7 +1,12 @@
 <?xml version="1.0"?>
 <robot xmlns:xacro="http://www.ros.org/wiki/xacro"  name="robot">
+    <xacro:arg name = "use_ros2_control" default="true"/>
     <xacro:include filename="robot_core.xacro"/>
-    <!-- <xacro:include filename="gazebo_control.xacro"/> -->
-    <xacro:include filename="ros2_control.xacro"/>
+    <xacro:if value = "$(arg use_ros2_control)">
+        <xacro:include filename="ros2_control.xacro"/>
+    </xacro:if>
+    <xacro:unless value = "$(arg use_ros2_control)">
+        <xacro:include filename="gazebo_control.xacro"/>
+    </xacro:unless>
     <xacro:include filename="lidar.xacro"/>
 </robot>

File: description/robot_core.xacro (robot description, xacro)
@@ -20,4 +20,12 @@
     <link name = "base_link">
     </link>
+    <!-- Base foot print -->
+     <joint name="base_footprint_joint" type="fixed">
+        <parent link="base_link"/>
+        <child link = "base_footprint"/>
+        <origin xyz = "0 0 0" rpy="0 0 0"/>
+     </joint>
+     <link name="base_footprint">
+     </link>
     <!-- Chassis -->
     <joint name = "chassis_joint" type="fixed">
